File: PCB/Drum.kicad_sch (KiCad schematic)
At the start: 3 parts, among them J1 Conn_01x08, U1 XIAO_ESP32_S3, U2 adafruit-MAX98357

Commit message: Finalized PCB designs
Parts:
- added H1, H2, H3, H4, H5: MountingHole, MountingHole:MountingHole_3.2mm_M3, symbol Mechanical:MountingHole
- J1: footprint (none) -> drumset:Drum buttons
